File: hub_1.kicad_sch (KiCad schematic)
At the start: 51 parts, among them J4 USB_C_Receptacle_USB2.0_16P, J5 USB_C_Receptacle_USB2.0_16P, J6 Header 01x04 0.1", U1 USBLC6-2P6, U2 USBLC6-2P6, U3 USBLC6-2P6, U4 USB2514B-I/M2, U5 MIC2026-1xM, U6 MIC2026-1xM, Y2 24MHz

Commit message: Updated for single USB line
Parts:
- removed C20, C21: 27pF, Capacitor_SMD:C_0603_1608Metric, symbol Device:C_Small
- removed C22, C25, C26, C27, C28, C29, C30, C36, C38: 0.1uF, Capacitor_SMD:C_0603_1608Metric, symbol Device:C_Small
- removed C23: 4.7uF, Capacitor_SMD:C_0603_1608Metric, symbol Device:C_Small
- removed C24: 1uF, Capacitor_SMD:C_0603_1608Metric, symbol Device:C_Small
- removed C37: 100uF, Capacitor_SMD:C_0805_2012Metric, symbol Device:C_Small
- removed D3: Green, LED_SMD:LED_0603_1608Metric, symbol Device:LED_Small
- removed FB3: 600R, Inductor_SMD:L_0603_1608Metric, symbol Device:FerriteBead_Small
- removed FL3: 744230900, CameraHub:CHIP_230900_WRE, symbol Filter:Choke_Wurth_WE-CNSW_744232090
- removed J6: Header 01x04 0.1", Connector_PinHeader_2.54mm:PinHeader_1x04_P2.54mm_Vertical, symbol Connector_Generic:Conn_01x04
- removed R10, R15, R24, R26: 36K, Resistor_SMD:R_0603_1608Metric, symbol Device:R_Small
- removed R19: 330R, Resistor_SMD:R_0603_1608Metric, symbol Device:R_Small
- removed R25: 12K, Resistor_SMD:R_0603_1608Metric, symbol Device:R_Small
- removed R33: 10K, Resistor_SMD:R_0603_1608Metric, symbol Device:R_Small
- removed R8: 1M, Resistor_SMD:R_0603_1608Metric, symbol Device:R_Small
- removed R9: 100K, Resistor_SMD:R_0603_1608Metric, symbol Device:R_Small
- removed U3: USBLC6-2P6, Package_TO_SOT_SMD:SOT-23-6, symbol Power_Protection:USBLC6-2P6
- removed U4: USB2514B-I/M2, Package_DFN_QFN:QFN-36-1EP_6x6mm_P0.5mm_EP3.7x3.7mm, symbol Interface_USB:USB2514B_Bi
- removed U6: MIC2026-1xM, Package_SO:SOIC-8_3.9x4.9mm_P1.27mm, symbol Power_Management:MIC2026-1xM
- removed Y2: 24MHz, Crystal:Crystal_SMD_3225-4Pin_3.2x2.5mm, symbol Device:Crystal_GND24_Small
Connections:
- no-connect marks 18 -> 8
