File: hub_2.kicad_sch (KiCad schematic)
At the start: 51 parts, among them J7 USB_C_Receptacle_USB2.0_16P, J8 USB_C_Receptacle_USB2.0_16P, J9 Header 01x04 0.1", U10 USB2514B-I/M2, U11 MIC2026-1xM, U12 MIC2026-1xM, U7 USBLC6-2P6, U8 USBLC6-2P6, U9 USBLC6-2P6, Y1 24MHz

Commit message: Updated for single USB line
Parts:
- removed FB6: 600R, Inductor_SMD:L_0603_1608Metric, symbol Device:FerriteBead_Small
- removed J9: Header 01x04 0.1", Connector_PinHeader_2.54mm:PinHeader_1x04_P2.54mm_Vertical, symbol Connector_Generic:Conn_01x04
- added C18: 100uF, Capacitor_SMD:C_0805_2012Metric, symbol Device:C_Small
- added C19: 0.1uF, Capacitor_SMD:C_0603_1608Metric, symbol Device:C_Small
- added D4: Green, LED_SMD:LED_0603_1608Metric, symbol Device:LED_Small
- added FB3, FB4: 600R, Inductor_SMD:L_0603_1608Metric, symbol Device:FerriteBead_Small
- added FL4: 744230900, CameraHub:CHIP_230900_WRE, symbol Filter:Choke_Wurth_WE-CNSW_744232090
- added J3, J4: USB_C_Receptacle_USB2.0_16P, CameraHub:USBC-121SMT-4BS2S, symbol Connector:USB_C_Receptacle_USB2.0_16P
- added R11: 10K, Resistor_SMD:R_0603_1608Metric, symbol Device:R_Small
- added R15: 330R, Resistor_SMD:R_0603_1608Metric, symbol Device:R_Small
- added U4: USBLC6-2P6, Package_TO_SOT_SMD:SOT-23-6, symbol Power_Protection:USBLC6-2P6
- renumbered C18 to C20, C19 to C21, D4 to D1, D5 to D2, D6 to D3, FB2 to FB1, FB5 to FB2, FL4 to FL1, FL5 to FL2, FL6 to FL3, J7 to J1, J8 to J2, R16 to R10, R20 to R12, R21 to R13, R22 to R14, R7 to R6, R6 to R7, R11 to R8, R12 to R9, U7 to U1, U8 to U2, U9 to U3, U10 to U5, U11 to U6, U12 to U7
Connections:
- net +3.3V: now also R11.1
- net D3_N: now also J3.A7 (D-), J3.B7 (D-)
- net D3_P: now also J3.A6 (D+), J3.B6 (D+)
- net GND: now also C18.2, C19.2, D4.1 (K), J3.A1 (GND), J3.A12 (GND), J3.B1 (GND), J3.B12 (GND), J3.S1 (SHIELD), J4.A1 (GND), J4.A12 (GND), J4.B1 (GND), J4.B12 (GND), J4.S1 (SHIELD), U4.2 (GND)
- net VBUS3: now also FB3.1
- net VBUS_CONN3: now also FB3.2, J3.A4 (VBUS), J3.A9 (VBUS), J3.B4 (VBUS), J3.B9 (VBUS)
- net PWR4: now reaches U5.20 (PRTPWR4/BC_EN4)
- net PWR4: now also U7.4 (ENB)
- net nOCS4: now reaches U5.21 (OCS_N4)
- net nOCS4: now also U7.3 (FLGB), R11.2
- net HD4_N: now reaches U5.8 (USBDM_DN4/PRT_DIS_M4)
- net HD4_N: now also FL4.4
- net HD4_P: now reaches U5.9 (USBDP_DN4/PRT_DIS_P4)
- net HD4_P: now also FL4.1
- net VBUS4: now reaches U7.5 (OUTB)
- net VBUS4: now also C18.1, C19.1, FB4.1
- new net: D4.2 (A), R15.2
- new net D4_N: J4.A7 (D-), J4.B7 (D-), U4.4 (I/O2)
- new net D4_P: J4.A6 (D+), J4.B6 (D+), U4.6 (I/O1)
- new net FD4_N: FL4.3, U4.3 (I/O2)
- new net FD4_P: FL4.2, U4.1 (I/O1)
- new net VBUS_CONN4: FB4.2, J4.A4 (VBUS), J4.A9 (VBUS), J4.B4 (VBUS), J4.B9 (VBUS), R15.1, U4.5 (VBUS)
- no-connect marks 18 -> 19
Other:
- moved on the sheet: C12, C13, C14, C15, C16, C17, C20, C21, D1, D2, D3, FL3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
